Commit message: - 在上位机 	- 更新URDF，添加左右两个轮子（后续可以换成以前自己建的fishbot urdf），添加可视旋转色标和 Gazebo 同步插件 	- 默认关闭测试用 joint_state_publisher，避免和 ESP32 同时发布 	- 新建launch，一键启动真机 bringup、Gazebo （零重力环境）和模型 - 在小车源码： 	- 添加函数 `float Kinematics::get_motor_distance`，用于获取已经行走的距离 	- 发布  joint_states

File: src/fishbot_description/urdf/fishbot.urdf (robot description, URDF)
Before this commit: robot fishbot, 3 links, 2 joints
Links:
- added link left_wheel_link, mass 0.05; collision cylinder length=0.04 radius=0.032; visual box size=0.050 0.004 0.006
- added link right_wheel_link, mass 0.05; collision cylinder length=0.04 radius=0.032; visual box size=0.050 0.004 0.006
- link base_link: mass None -> 2.0; geometry collision cylinder length=0.12 radius=0.10; visual cylinder length=0.12 radius=0.10
- link laser_link: mass None -> 0.05; geometry collision cylinder length=0.02 radius=0.02; visual cylinder length=0.02 radius=0.02
Joints:
- added joint left_wheel_joint: type continuous, parent base_link, child left_wheel_link, origin xyz=-0.02 0.10 -0.044 rpy=0 0 0, axis 0 -1 0, limit effort=2.0 velocity=100.0
- added joint right_wheel_joint: type continuous, parent base_link, child right_wheel_link, origin xyz=-0.02 -0.10 -0.044 rpy=0 0 0, axis 0 -1 0, limit effort=2.0 velocity=100.0
